File: Apple M0110.sch (KiCad schematic (older format))
At the start: 132 parts, among them J1 SW_PUSH, K1 SW_PUSH, M1 SW_PUSH, P1 SW_PUSH, Q1 SW_PUSH, T1 SW_PUSH, U1 SW_PUSH, X1 SW_PUSH, Y1 SW_PUSH

Commit message: Replace the MX only footprints with Alps + MX switch footprints
Parts:
- A1, B1, BACK_SLSH1, C1, COMMA1, D18, DASH1, E1, EQUALS1, ESC1, F1, FWD_SLSH1, G1, H1, I1, J1, K1, L1, LEFT_BRKT1, L_ALT1, L_ALT3, L_CMD1, L_FN_ALT2, M1, N1, NUM_ROW_0, NUM_ROW_1, NUM_ROW_2, NUM_ROW_3, NUM_ROW_4, NUM_ROW_5, NUM_ROW_6, NUM_ROW_7, NUM_ROW_8, NUM_ROW_9, O1, P1, PERIOD1, Q1, QUOTE1, R1, RGHT_BRKT1, R_ALT1, R_ALT3, R_CMD1, S1, SEMI_COLON1, T1, TAB1, U1, V1, W1, X1, Y1, Z1: footprint keyboard_footprints:MX_PCB_100H -> saucy_footprints:Hybrid_PCB_LED_100H
- BACKSPACE1, R_CMD2, R_CMD3, R_FN_ALT2: footprint keyboard_footprints:MX_PCB_150H -> saucy_footprints:Hybrid_PCB_LED_100H
- CAPS_LOCK1, ENTER1: footprint keyboard_footprints:MX_PCB_175H -> saucy_footprints:Hybrid_PCB_175H
- L_CMD2, L_CMD3: footprint keyboard_footprints:MX_PCB_150H -> saucy_footprints:MX_PCB_100H
- L_SHIFT1, R_SHIFT1: footprint keyboard_footprints:MX_PCB_225H -> saucy_footprints:Hybrid_PCB_LED_225H
